File: kicad-2/jjrpulser.kicad_pcb (KiCad board)
At the start: 2 copper layers, 32.8 x 43.5 mm, 27 parts, among them J1 5V Input, J2 Hot&Cold Terminal, J5 Conn_UART, U1 ESP-12, U2 AMS1117-3.3_SOT223

Commit message: Новая разводка: буквы и размеры
Other:
- board text added: "+"
- board text added: "-"
- board text added: "COLD"
- board text added: "GND"
- board text added: "GREEN"
- board text added: "HOT"
- board text added: "JJR"
- board text added: "RED"
- board text added: "RTS"
Changed lines of the file:
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@@
     (links 46)
     (no_connects 0)
-    (area 139.174999 86.174999 172.075001 129.825001)
+    (area 136.889993 82.824999 186.992858 140.200001)
     (thickness 1.6)
-    (drawings 4)
+    (drawings 15)
     (tracks 108)
     (zones 0)
@@
     (38 B.Mask user)
     (39 F.Mask user)
+    (40 Dwgs.User user)
+    (41 Cmts.User user)
     (44 Edge.Cuts user)
     (45 Margin user)
@@
     (user_trace_width 2)
     (trace_clearance 0.1)
-    (zone_clearance 0.508)
+    (zone_clearance 0.5)
     (zone_45_only no)
     (trace_min 0.3)
@@
     )
   )
+  (dimension 43.5 (width 0.3) (layer Cmts.User)
+    (gr_text "43,5 мм" (at 182.35 108 270) (layer Cmts.User)
+      (effects (font (size 1.5 1.5) (thickness 0.3)))
+    )
+    (feature1 (pts (xy 172 129.75) (xy 183.7 129.75)))
+    (feature2 (pts (xy 172 86.25) (xy 183.7 86.25)))
+    (crossbar (pts (xy 181 86.25) (xy 181 129.75)))
+    (arrow1a (pts (xy 181 129.75) (xy 180.413579 128.623496)))
+    (arrow1b (pts (xy 181 129.75) (xy 181.586421 128.623496)))
+    (arrow2a (pts (xy 181 86.25) (xy 180.413579 87.376504)))
+    (arrow2b (pts (xy 181 86.25) (xy 181.586421 87.376504)))
+  )
+  (dimension 32.75 (width 0.3) (layer Cmts.User)
+    (gr_text "32,75 мм" (at 155.625 138.85) (layer Cmts.User)
+      (effects (font (size 1.5 1.5) (thickness 0.3)))
+    )
+    (feature1 (pts (xy 172 129.75) (xy 172 140.2)))
+    (feature2 (pts (xy 139.25 129.75) (xy 139.25 140.2)))
+    (crossbar (pts (xy 139.25 137.5) (xy 172 137.5)))
+    (arrow1a (pts (xy 172 137.5) (xy 170.873496 138.086421)))
+    (arrow1b (pts (xy 172 137.5) (xy 170.873496 136.913579)))
+    (arrow2a (pts (xy 139.25 137.5) (xy 140.376504 138.086421)))
+    (arrow2b (pts (xy 139.25 137.5) (xy 140.376504 136.913579)))
+  )
+  (gr_text RED (at 140 109.5 270) (layer B.Cu)
+    (effects (font (size 1 1) (thickness 0.25)) (justify mirror))
+  )
+  (gr_text GREEN (at 142 123) (layer B.Cu)
+    (effects (font (size 1 1) (thickness 0.25)) (justify mirror))
+  )
+  (gr_text JJR (at 142.5 128) (layer B.Cu)
+    (effects (font (size 2 2) (thickness 0.5) italic) (justify mirror))
+  )
+  (gr_text - (at 164.5 128) (layer B.Cu)
+    (effects (font (size 2 2) (thickness 0.5)) (justify mirror))
+  )
+  (gr_text + (at 159.5 128) (layer B.Cu)
+    (effects (font (size 2 2) (thickness 0.5)) (justify mirror))
+  )
+  (gr_text GND (at 159 88) (layer B.Cu)
+    (effects (font (size 2 2) (thickness 0.5)) (justify mirror))
+  )
+  (gr_text RTS (at 148 88) (layer B.Cu)
+    (effects (font (size 2 2) (thickness 0.5)) (justify mirror))
+  )
+  (gr_text HOT (at 170.5 102.5 90) (layer B.Cu)
+    (effects (font (size 2 2) (thickness 0.5)) (justify mirror))
+  )
+  (gr_text COLD (at 170.5 118 90) (layer B.Cu)
+    (effects (font (size 2 2) (thickness 0.5)) (justify mirror))
+  )
   (gr_line (start 139.25 86.25) (end 139.25 129.75) (angle 90) (layer Edge.Cuts) (width 0.15))
